File: MBP 15 Inch A1286 Upgrade/MBP 15 Inch A1286 Upgrade.sch (KiCad schematic (older format))
At the start: 3 parts, among them J1 501745-0301, J3401 500913-0302, P1 AdapterPCIEContacts

Commit message: Added 15-inch 1st revision
Other:
- note added: "The part featured here is a connector \nfrom Molex. Part number is listed\nunder net label. This is not part of the \nadapter, it is for reference."
- note removed: "The part featured here is a connector \nfrom Mouser. Part number is listed\nunder net label. This is not part of the \nadapter, it is for reference."
Changed lines of the file:
@@
 Unibody MacBook Logic Board Connector:
 Text Notes 700  5350 0    50   ~ 0
-The part featured here is a connector \nfrom Mouser. Part number is listed\nunder net label. This is not part of the \nadapter, it is for reference.
+The part featured here is a connector \nfrom Molex. Part number is listed\nunder net label. This is not part of the \nadapter, it is for reference.
 Wire Wire Line
 	1550 2800 1450 2800
