File: MBP 17 Inch A1297 2010-11 Upgrade/MBP 17 Inch A1297 Upgrade.kicad_pcb (KiCad board)
At the start: 2 copper layers, 27.8 x 29.9 mm, 4 parts, among them J1 501745-0301

Commit message: Deleted temporary files and added images
Parts:
- moved REF** 2.01 mm to (99.3, 47.5)
Other:
- board text added: "MacBook 17 inch"
- board text removed: "21 - 25mm imac"
- board text removed: "MacBook 15in 2009 only"
Changed lines of the file:
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@@
   (general
     (thickness 1.6)
-    (drawings 15)
+    (drawings 14)
     (tracks 149)
     (zones 0)
@@
       (effects (font (size 1.27 1.27) (thickness 0.254)))
     )
+    (fp_line (start -4 -1.319) (end -4 0.811) (layer F.SilkS) (width 0.1))
+    (fp_line (start 4 -1.319) (end 4 0.811) (layer F.SilkS) (width 0.1))
+    (fp_line (start 5 2.511) (end 5 -3.019) (layer F.CrtYd) (width 0.1))
+    (fp_line (start -5 2.511) (end 5 2.511) (layer F.CrtYd) (width 0.1))
+    (fp_line (start -5 -3.019) (end -5 2.511) (layer F.CrtYd) (width 0.1))
+    (fp_line (start 5 -3.019) (end -5 -3.019) (layer F.CrtYd) (width 0.1))
+    (fp_line (start 4 0.811) (end 4 -1.319) (layer F.Fab) (width 0.2))
+    (fp_line (start -4 0.811) (end 4 0.811) (layer F.Fab) (width 0.2))
+    (fp_line (start -4 -1.319) (end -4 0.811) (layer F.Fab) (width 0.2))
     (fp_line (start 4 -1.319) (end -4 -1.319) (layer F.Fab) (width 0.2))
-    (fp_line (start -4 -1.319) (end -4 0.811) (layer F.Fab) (width 0.2))
-    (fp_line (start -4 0.811) (end 4 0.811) (layer F.Fab) (width 0.2))
-    (fp_line (start 4 0.811) (end 4 -1.319) (layer F.Fab) (width 0.2))
-    (fp_line (start 5 -3.019) (end -5 -3.019) (layer F.CrtYd) (width 0.1))
-    (fp_line (start -5 -3.019) (end -5 2.511) (layer F.CrtYd) (width 0.1))
-    (fp_line (start -5 2.511) (end 5 2.511) (layer F.CrtYd) (width 0.1))
-    (fp_line (start 5 2.511) (end 5 -3.019) (layer F.CrtYd) (width 0.1))
-    (fp_line (start 4 -1.319) (end 4 0.811) (layer F.SilkS) (width 0.1))
-    (fp_line (start -4 -1.319) (end -4 0.811) (layer F.SilkS) (width 0.1))
     (fp_text user %R (at 0 -0.254) (layer F.Fab)
       (effects (font (size 1.27 1.27) (thickness 0.254)))
@@
       (effects (font (size 1 1) (thickness 0.15)))
     )
+    (fp_circle (center 0 0) (end 2.75 0) (layer F.CrtYd) (width 0.05))
+    (fp_circle (center 0 0) (end 2.5 0) (layer Cmts.User) (width 0.15))
     (fp_text user %R (at 0.3 0) (layer F.Fab)
       (effects (font (size 1 1) (thickness 0.15)))
     )
-    (fp_circle (center 0 0) (end 2.5 0) (layer Cmts.User) (width 0.15))
-    (fp_circle (center 0 0) (end 2.75 0) (layer F.CrtYd) (width 0.05))
     (pad 1 thru_hole circle (at 0 0) (size 4 4) (drill 2.5) (layers *.Cu *.Mask))
   )
   (module "MBPWirelessUpgrade:MacBook Air Wireless Card" (layer F.Cu)
-    (at 99.2886 45.4914)
+    (at 99.2886 47.498)
     (fp_text reference REF** (at 13.708 17.018 90) (layer F.SilkS)
       (effects (font (size 1 1) (thickness 0.15)))
@@
       (effects (font (size 1 1) (thickness 0.15)))
     )
+    (fp_line (start 7.099 34.952) (end 7.099 37.665) (layer Edge.Cuts) (width 0.1))
+    (fp_line (start 6.333 34.952) (end 6.333 37.665) (layer Edge.Cuts) (width 0.1))
+    (fp_line (start 7.349 38) (end 7.099 37.665) (layer Edge.Cuts) (width 0.1))
+    (fp_line (start 7.349 38) (end 16.493 38) (layer Edge.Cuts) (width 0.1))
+    (fp_line (start 6.079 38) (end 6.329 37.665) (layer Edge.Cuts) (width 0.1))
+    (fp_line (start 1.507 38) (end 6.079 38) (layer Edge.Cuts) (width 0.1))
+    (fp_line (start 16.771 37.665) (end 16.493 38) (layer Edge.Cuts) (width 0.1))
+    (fp_line (start 16.771 34.444) (end 16.771 37.665) (layer Edge.Cuts) (width 0.1))
+    (fp_line (start 0.254 0) (end 7 0) (layer Edge.Cuts) (width 0.1))
+    (fp_line (start 1.229 37.665) (end 1.507 38) (layer Edge.Cuts) (width 0.1))
+    (fp_line (start 18 0.254) (end 18 33.274) (layer Edge.Cuts) (width 0.1))
+    (fp_line (start 11 0) (end 17.746 0) (layer Edge.Cuts) (width 0.1))
+    (fp_line (start 0 0.254) (end 0 33.274) (layer Edge.Cuts) (width 0.1))
+    (fp_line (start 16.771 34.444) (end 18 33.274) (layer Edge.Cuts) (width 0.1))
+    (fp_line (start 0 33.274) (end 1.229 34.444) (layer Edge.Cuts) (width 0.1))
     (fp_line (start 1.229 34.444) (end 1.229 37.665) (layer Edge.Cuts) (width 0.1))
-    (fp_line (start 0 33.274) (end 1.229 34.444) (layer Edge.Cuts) (width 0.1))
-    (fp_line (start 16.771 34.444) (end 18 33.274) (layer Edge.Cuts) (width 0.1))
-    (fp_line (start 0 0.254) (end 0 33.274) (layer Edge.Cuts) (width 0.1))
-    (fp_line (start 11 0) (end 17.746 0) (layer Edge.Cuts) (width 0.1))
-    (fp_line (start 18 0.254) (end 18 33.274) (layer Edge.Cuts) (width 0.1))
-    (fp_line (start 1.229 37.665) (end 1.507 38) (layer Edge.Cuts) (width 0.1))
-    (fp_line (start 0.254 0) (end 7 0) (layer Edge.Cuts) (width 0.1))
-    (fp_line (start 16.771 34.444) (end 16.771 37.665) (layer Edge.Cuts) (width 0.1))
-    (fp_line (start 16.771 37.665) (end 16.493 38) (layer Edge.Cuts) (width 0.1))
-    (fp_line (start 1.507 38) (end 6.079 38) (layer Edge.Cuts) (width 0.1))
-    (fp_line (start 6.079 38) (end 6.329 37.665) (layer Edge.Cuts) (width 0.1))
-    (fp_line (start 7.349 38) (end 16.493 38) (layer Edge.Cuts) (width 0.1))
-    (fp_line (start 7.349 38) (end 7.099 37.665) (layer Edge.Cuts) (width 0.1))
-    (fp_line (start 6.333 34.952) (end 6.333 37.665) (layer Edge.Cuts) (width 0.1))
-    (fp_line (start 7.099 34.952) (end 7.099 37.665) (layer Edge.Cuts) (width 0.1))
     (fp_text user "MacBook Air Wireless Card" (at 8.89 18.288 90) (layer B.SilkS)
       (effects (font (size 1.5 1.5) (thickness 0.15)) (justify mirror))
@@
   (module "" (layer F.Cu)
     (at 108.602 88.6595)
-    (fp_text reference P1 (at 8.0518 2.667) (layer F.SilkS)
+    (fp_text reference P1 (at -1.414 3.0345) (layer F.SilkS)
       (effects (font (size 1.27 1.27) (thickness 0.15)))
     )
@@
   )
   (gr_line (start 119.2276 86.106) (end 119.2276 70.1294) (layer Edge.Cuts) (width 0.1))
-  (gr_text "MacBook 15in 2009 only" (at 119.3546 90.5256 90) (layer F.SilkS)
+  (gr_text "MacBook 17 inch" (at 119.126 93.218 90) (layer F.SilkS)
     (effects (font (size 1 1) (thickness 0.15)))
   )
-  (gr_text "21 - 25mm imac" (at 128.6256 81.3816) (layer F.SilkS)
-    (effects (font (size 1 1) (thickness 0.15)))
-  )
